Commit message: Implement a direct force controller that uses KDL & change name of the package

File: panda_controllers/model/robots/sim.urdf (robot description, URDF)
Before this commit: robot lumi, 15 links, 14 joints
Links:
- link lumi_hand: mass None -> 0.68
- link lumi_leftfinger: mass None -> 0.01
- link lumi_link0: mass None -> 3.06
- link lumi_link1: mass None -> 2.34
- link lumi_link2: mass None -> 2.36
- link lumi_link3: mass None -> 2.38
- link lumi_link4: mass None -> 2.43
- link lumi_link5: mass None -> 3.5
- link lumi_link6: mass None -> 1.47
- link lumi_link7: mass None -> 0.45
- link lumi_link8: mass None -> 0.0
- link lumi_rightfinger: mass None -> 0.01

Commit message: Modelled friction for puck model and tested the result with force controller

File: panda_controllers/model/robots/sim.urdf (robot description, URDF)
Before this commit: robot lumi, 15 links, 14 joints
Links:
- added link hockeyPuck, mass 0.1; collision mesh filename=package://panda_controllers/model/meshes/hockeyPuck.stl scale=4.5 4.5 4.5; visual mesh filename=package://panda_controllers/model/meshes/hockeyPuck.stl scale=4.5 4.5 4.5
Joints:
- added joint puckjoint: type floating, parent base_link, child hockeyPuck, origin xyz=0.5 0 0 rpy=0 0 0
